File: kicad/kicad_slugtpu.kicad_sch (KiCad schematic)
At the start: 2 parts, among them U1 MT48LC16M16A2TG

Commit message: update kicad schematic
Parts:
- added U3: ESP32-C3-MINI-1-N4, ESP32-C3-MINI-1_EXP, symbol esp32-c3-mini-1-n4x:ESP32-C3-MINI-1-N4
- U2: value ~ -> TPU
Other:
- moved on the sheet: U1
Changed lines of the file:
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@@
 	(symbol
 		(lib_id "slugtpu:tpu")
-		(at 69.85 43.18 0)
+		(at 129.54 38.1 0)
 		(unit 1)
 		(exclude_from_sim no)
@@
 		(dnp no)
 		(property "Reference" "U2"
-			(at 67.818 43.688 0)
-			(effects
-				(font
-					(size 1.27 1.27)
-				)
-				(justify left)
-			)
-		)
-		(property "Value" "~"
-			(at 83.82 95.8849 0)
-			(effects
-				(font
-					(size 1.27 1.27)
-				)
-				(justify left)
+			(at 129.54 36.576 0)
+			(effects
+				(font
+					(size 1.27 1.27)
+				)
+			)
+		)
+		(property "Value" "TPU"
+			(at 129.54 39.37 0)
+			(effects
+				(font
+					(size 1.27 1.27)
+				)
 			)
 		)
 		(property "Footprint" ""
-			(at 69.85 43.18 0)
+			(at 129.54 38.1 0)
 			(effects
 				(font
@@
 		)
 		(property "Datasheet" ""
-			(at 69.85 43.18 0)
+			(at 129.54 38.1 0)
 			(effects
 				(font
@@
 		)
 		(property "Description" ""
-			(at 69.85 43.18 0)
+			(at 129.54 38.1 0)
 			(effects
 				(font
@@
 	)
 	(symbol
+		(lib_id "esp32-c3-mini-1-n4x:ESP32-C3-MINI-1-N4")
+		(at 35.56 34.29 0)
+		(unit 1)
+		(exclude_from_sim no)
+		(in_bom yes)
+		(on_board yes)
+		(dnp no)
+		(fields_autoplaced yes)
+		(property "Reference" "U3"
+			(at 55.88 24.13 0)
+			(effects
+				(font
+					(size 1.524 1.524)
+				)
+			)
+		)
+		(property "Value" "ESP32-C3-MINI-1-N4"
+			(at 55.88 26.67 0)
+			(effects
+				(font
+					(size 1.524 1.524)
+				)
+			)
+		)
+		(property "Footprint" "ESP32-C3-MINI-1_EXP"
+			(at 35.56 34.29 0)
+			(effects
+				(font
+					(size 1.27 1.27)
+					(italic yes)
+				)
+				(hide yes)
+			)
+		)
+		(property "Datasheet" "ESP32-C3-MINI-1-N4"
+			(at 35.56 34.29 0)
+			(effects
+				(font
+					(size 1.27 1.27)
+					(italic yes)
+				)
+				(hide yes)
+			)
+		)
+		(property "Description" ""
+			(at 35.56 34.29 0)
+			(effects
+				(font
+					(size 1.27 1.27)
+				)
+				(hide yes)
+			)
+		)
+		(pin "60"
+		)
+		(pin "51"
+		)
+		(pin "7"
+		)
+		(pin "49"
+		)
+		(pin "1"
+		)
+		(pin "39"
+		)
+		(pin "14"
+		)
+		(pin "4"
+		)
+		(pin "15"
+		)
+		(pin "8"
+		)
+		(pin "5"
+		)
+		(pin "6"
+		)
+		(pin "55"
+		)
+		(pin "2"
+		)
+		(pin "34"
+		)
+		(pin "48"
+		)
+		(pin "13"
+		)
+		(pin "37"
+		)
+		(pin "38"
+		)
+		(pin "18"
+		)
+		(pin "53"
+		)
+		(pin "27"
+		)
+		(pin "30"
+		)
+		(pin "31"
+		)
+		(pin "26"
+		)
+		(pin "58"
+		)
+		(pin "46"
+		)
+		(pin "24"
+		)
+		(pin "59"
+		)
+		(pin "28"
+		)
+		(pin "23"
+		)
+		(pin "54"
+		)
+		(pin "10"
+		)
+		(pin "61"
+		)
+		(pin "3"
+		)
+		(pin "17"
+		)
+		(pin "40"
+		)
+		(pin "35"
+		)
+		(pin "41"
+		)
+		(pin "42"
+		)
+		(pin "22"
+		)
+		(pin "47"
+		)
+		(pin "36"
+		)
+		(pin "44"
+		)
+		(pin "20"
+		)
+		(pin "32"
+		)
+		(pin "33"
+		)
+		(pin "25"
+		)
+		(pin "16"
+		)
+		(pin "21"
+		)
+		(pin "29"
+		)
+		(pin "19"
+		)
+		(pin "52"
+		)
+		(pin "45"
+		)
+		(pin "56"
+		)
+		(pin "11"
+		)
+		(pin "9"
+		)
+		(pin "12"
+		)
+		(pin "43"
+		)
+		(pin "50"
+		)
+		(pin "57"
+		)
+		(instances
+			(project "kicad_slugtpu"
+				(path "/4425e230-e1b9-48b0-8e28-a79ff0241594"
+					(reference "U3")
+					(unit 1)
+				)
+			)
+		)
+	)
+	(symbol
 		(lib_id "Memory_RAM:MT48LC16M16A2TG")
-		(at 207.01 95.25 0)
+		(at 232.41 72.39 0)
 		(unit 1)
 		(exclude_from_sim no)
@@
 		(fields_autoplaced yes)
 		(property "Reference" "U1"
-			(at 209.1533 57.15 0)
+			(at 234.5533 34.29 0)
 			(effects
 				(font
@@
 		)
 		(property "Value" "MT48LC16M16A2TG"
-			(at 209.1533 59.69 0)
+			(at 234.5533 36.83 0)
 			(effects
 				(font
@@
 		)
 		(property "Footprint" "Package_SO:TSOP-II-54_22.2x10.16mm_P0.8mm"
-			(at 207.01 130.81 0)
+			(at 232.41 107.95 0)
 			(effects
 				(font
@@
 		)
 		(property "Datasheet" "https://www.micron.com/-/media/client/global/documents/products/data-sheet/dram/256mb_sdr.pdf"
-			(at 207.01 101.6 0)
+			(at 232.41 78.74 0)
 			(effects
 				(font
@@
 		)
 		(property "Description" "256M – (16M x 16 bit) Synchronous DRAM (SDRAM), TSOP-II-54"
-			(at 207.01 95.25 0)
-			(effects
-				(font
+			(at 232.41 72.39 0)
+			(effects
+				(font
